Commit message: Format test.xacro

File: ros/catkin_ws/src/david_config/urdf/test.xacro (robot description, xacro)
@@ -3,9 +3,9 @@
   <link name="base_link" />
   <link name="map" />
-  <joint name"d455_2_link" type="fixed">
-      <origin rpy="0 0 0" xyz="0 0 0"/>
-      <parent link="map"/>
-      <child link="base_link"/>
-      <axis xyz="0 0 0"/>
+  <joint name="d455_2_link" type="fixed">
+    <origin rpy="0 0 0" xyz="0 0 0"/>
+    <parent link="map" />
+    <child link="base_link" />
+    <axis xyz="0 0 0" />
   </joint>
 </robot>

Commit message: Update test.xacro

File: ros/catkin_ws/src/david_config/urdf/test.xacro (robot description, xacro)
@@ -1,11 +1,25 @@
 <?xml version="1.0" ?>
 <robot name="david" xmlns:xacro="http://www.ros.org/wiki/xacro" >
-  <link name="base_link" />
-  <link name="map" />
-  <joint name="d455_2_link" type="fixed">
-    <origin rpy="0 0 0" xyz="0 0 0"/>
-    <parent link="map" />
-    <child link="base_link" />
-    <axis xyz="0 0 0" />
-  </joint>
+    <link name="base_link" />
+    <link name="map" />
+    <joint name="stationary_robot" type="fixed">
+        <origin rpy="0 0 0" xyz="0 0 0"/>
+        <parent link="map" />
+        <child link="base_link" />
+        <axis xyz="0 0 0" />
+    </joint>
+    <link name="d455_2_link" />
+    <link name="t265_link" />
+    <joint name="d455_2_joint" type="fixed">
+        <origin rpy="0 0 0" xyz="0 0.199 0" />
+        <parent link="base_link" />
+        <child link="d455_2_link" />
+        <axis xyz="0 0 0" />
+    </joint>
+    <joint name="t265_joint" type="fixed">
+        <origin rpy="0 0 0" xyz="0.0131 0.068 0" />
+        <parent link="base_link" />
+        <child link="t265_link" />
+        <axis xyz="0 0 0" />
+    </joint>
 </robot>

Commit message: some stuff

File: ros/catkin_ws/src/david_config/urdf/test.xacro (robot description, xacro)
@@ -1,15 +1,22 @@
 <?xml version="1.0" ?>
 <robot name="david" xmlns:xacro="http://www.ros.org/wiki/xacro" >
+    <link name="base_link" />
     <link name="d455_2_link" />
     <link name="t265_link" />
     <link name="t265_pose_frame" />
+    <!-- Base link should be center of robot -->
+    <joint name="base_joint">
+        <origin rpy="0 0 0" xyz="0 0 0" />
+        <parent link="t265_pose_frame" />
+        <child link="base_link" />
+    </joint>
     <joint name="d455_2_joint" type="fixed">
         <origin rpy="3.14 0 0" xyz="0 0.199 0" />
-        <parent link="t265_pose_frame" />
+        <parent link="base_link" />
         <child link="d455_2_link" />
     </joint>
     <joint name="t265_joint" type="fixed">
         <origin rpy="0 0 0" xyz="0.0131 0.068 0" />
-        <parent link="t265_pose_frame" />
+        <parent link="base_link" />
         <child link="t265_link" />
     </joint>

Commit message: urdf stuff

File: ros/catkin_ws/src/david_config/urdf/test.xacro (robot description, xacro)
@@ -1,8 +1,15 @@
 <?xml version="1.0" ?>
 <robot name="david" xmlns:xacro="http://www.ros.org/wiki/xacro" >
+    <link name="map" />
     <link name="base_link" />
     <link name="d455_2_link" />
     <link name="t265_link" />
     <link name="t265_pose_frame" />
+    <link name="t265_odom_frame" />
+    <joint name="map_joint">
+        <origin rpy="0 0 0" xyz="0 0 0" />
+        <parent link="map" />
+        <child link="t265_odom_frame" />
+    </joint>
     <!-- Base link should be center of robot -->
     <joint name="base_joint">

Commit message: Small updates

File: ros/catkin_ws/src/david_config/urdf/test.xacro (robot description, xacro)
@@ -7,9 +7,4 @@
     <link name="t265_pose_frame" />
     <link name="t265_odom_frame" />
-    <joint name="map_joint">
-        <origin rpy="0 0 0" xyz="0 0 0" />
-        <parent link="map" />
-        <child link="t265_odom_frame" />
-    </joint>
     <!-- Base link should be center of robot -->
     <joint name="base_joint">
