Commit message: mapping works

File: ros/catkin_ws/src/david_config/urdf/test.urdf (robot description, URDF)
Before this commit: robot david, 4 links, 3 joints
Links:
- removed link base_link
- removed link map
- added link t265_pose_frame
Joints:
- removed joint stationary_robot
- joint d455_2_joint: axis 0 0 0 -> (none); origin xyz=0 0.199 0 rpy=0 0 0 -> xyz=0 0.199 0 rpy=3.14 0 0; parent base_link -> t265_pose_frame
- joint t265_joint: axis 0 0 0 -> (none); parent base_link -> t265_pose_frame

File: ros/catkin_ws/src/david_config/urdf/test.xacro (robot description, xacro)
@@ -1,25 +1,16 @@
 <?xml version="1.0" ?>
 <robot name="david" xmlns:xacro="http://www.ros.org/wiki/xacro" >
-    <link name="base_link" />
-    <link name="map" />
-    <joint name="stationary_robot" type="fixed">
-        <origin rpy="0 0 0" xyz="0 0 0"/>
-        <parent link="map" />
-        <child link="base_link" />
-        <axis xyz="0 0 0" />
-    </joint>
     <link name="d455_2_link" />
     <link name="t265_link" />
+    <link name="t265_pose_frame" />
     <joint name="d455_2_joint" type="fixed">
-        <origin rpy="0 0 0" xyz="0 0.199 0" />
-        <parent link="base_link" />
+        <origin rpy="3.14 0 0" xyz="0 0.199 0" />
+        <parent link="t265_pose_frame" />
         <child link="d455_2_link" />
-        <axis xyz="0 0 0" />
     </joint>
     <joint name="t265_joint" type="fixed">
         <origin rpy="0 0 0" xyz="0.0131 0.068 0" />
-        <parent link="base_link" />
+        <parent link="t265_pose_frame" />
         <child link="t265_link" />
-        <axis xyz="0 0 0" />
     </joint>
 </robot>

Commit message: stuff

File: ros/catkin_ws/src/david_config/urdf/test.urdf (robot description, URDF)
Before this commit: robot david, 3 links, 2 joints
Links:
- added link base_link
Joints:
- added joint base_joint: type fixed, parent t265_pose_frame, child base_link, origin xyz=0 0 0 rpy=0 0 0
- joint d455_2_joint: parent t265_pose_frame -> base_link
- joint t265_joint: parent t265_pose_frame -> base_link

File: ros/catkin_ws/src/david_config/urdf/test.xacro (robot description, xacro)
@@ -1,12 +1,10 @@
 <?xml version="1.0" ?>
 <robot name="david" xmlns:xacro="http://www.ros.org/wiki/xacro" >
-    <link name="map" />
     <link name="base_link" />
     <link name="d455_2_link" />
     <link name="t265_link" />
     <link name="t265_pose_frame" />
-    <link name="t265_odom_frame" />
     <!-- Base link should be center of robot -->
-    <joint name="base_joint">
+    <joint name="base_joint" type="fixed">
         <origin rpy="0 0 0" xyz="0 0 0" />
         <parent link="t265_pose_frame" />

Commit message: testing mapping

File: ros/catkin_ws/src/david_config/urdf/test.urdf (robot description, URDF)
Before this commit: robot david, 4 links, 3 joints
Links:
- removed link d455_2_link
- added link l515_1_link
Joints:
- removed joint d455_2_joint
- added joint l515_1_joint: type fixed, parent base_link, child l515_1_link, origin xyz=-0.03 0 0 rpy=0 0 0
- joint t265_joint: origin xyz=0.0131 0.068 0 rpy=0 0 0 -> xyz=0 0 0 rpy=0 0 0

File: ros/catkin_ws/src/david_config/urdf/test.xacro (robot description, xacro)
@@ -2,5 +2,5 @@
 <robot name="david" xmlns:xacro="http://www.ros.org/wiki/xacro" >
     <link name="base_link" />
-    <link name="d455_2_link" />
+    <link name="l515_1_link" />
     <link name="t265_link" />
     <link name="t265_pose_frame" />
@@ -11,11 +11,11 @@
         <child link="base_link" />
     </joint>
-    <joint name="d455_2_joint" type="fixed">
-        <origin rpy="3.14 0 0" xyz="0 0.199 0" />
+    <joint name="l515_1_joint" type="fixed">
+        <origin rpy="0 0 0" xyz="-0.03 0 0" />
         <parent link="base_link" />
-        <child link="d455_2_link" />
+        <child link="l515_1_link" />
     </joint>
     <joint name="t265_joint" type="fixed">
-        <origin rpy="0 0 0" xyz="0.0131 0.068 0" />
+        <origin rpy="0 0 0" xyz="0 0 0" />
         <parent link="base_link" />
         <child link="t265_link" />
