Commit message: Fix david2.urdf

File: ros/catkin_ws/src/david_config/urdf/david2.urdf (robot description, URDF)
Before this commit: robot david, 10 links, 9 joints
Joints:
- removed joint None
- added joint l515_1_joint: type fixed, parent left_tread, child l515_1, origin xyz=0.45 -0.04 0.38, axis 0 0 0
- joint back_right_joint: type None -> fixed
- joint back_sensor_joint: type None -> fixed
- joint d455_1_joint: type None -> fixed
- joint d455_2_joint: type None -> fixed
- joint l515_2_joint: origin xyz=-0.045 0 0.185 rpy=0 10 0 -> xyz=-0.045 0 0.185 rpy=0 -0.1745329252 0; type None -> fixed
- joint left_tread_joint: type None -> fixed
- joint right_tread_joint: type None -> fixed
- joint t265_joint: type None -> fixed

Commit message: Slopes on cameras

File: ros/catkin_ws/src/david_config/urdf/david2.urdf (robot description, URDF)
Before this commit: robot david, 10 links, 9 joints
Joints:
- joint d455_1_joint: origin xyz=-0.005 -0.02 0.16 -> xyz=-0.005 -0.02 0.16 rpy=-0.261799387799 0 0
- joint d455_2_joint: origin xyz=-0.01 0.02 0.16 rpy=0 0 0 -> xyz=-0.01 0.02 0.16 rpy=0.261799387799 0 0
- joint l515_1_joint: origin xyz=0.45 -0.04 0.38 -> xyz=0.45 -0.04 0.38 rpy=0 0.261799387799 0

Commit message: Update transforms for cameras

File: ros/catkin_ws/src/david_config/urdf/david2.urdf (robot description, URDF)
Before this commit: robot david, 10 links, 9 joints
Joints:
- joint d455_1_joint: origin xyz=-0.005 -0.02 0.16 rpy=-0.261799387799 0 0 -> xyz=-0.005 -0.02 0.16 rpy=-1.8325957146 0 0
- joint d455_2_joint: origin xyz=-0.01 0.02 0.16 rpy=0.261799387799 0 0 -> xyz=-0.01 0.02 0.16 rpy=1.308996939 3.14159265 0

Commit message: Update URDF link names

File: ros/catkin_ws/src/david_config/urdf/david2.urdf (robot description, URDF)
Before this commit: robot david, 10 links, 9 joints
Links:
- removed link d455_1
- removed link d455_2
- removed link l515_1
- removed link l515_2
- removed link t265
- added link d455_1_link
- added link d455_2_link
- added link l515_1_link
- added link l515_2_link
- added link t265_link
Joints:
- removed joint d455_1_joint
- removed joint d455_2_joint
- removed joint l515_1_joint
- removed joint l515_2_joint
- removed joint t265_joint
- added joint d455_1_link_joint: type fixed, parent left_tread, child d455_1_link, origin xyz=-0.005 -0.02 0.16 rpy=-1.8325957146 0 0, axis 0 0 0
- added joint d455_2_link_joint: type fixed, parent right_tread, child d455_2_link, origin xyz=-0.01 0.02 0.16 rpy=1.308996939 3.14159265 0, axis 0 0 0
- added joint l515_1_link_joint: type fixed, parent left_tread, child l515_1_link, origin xyz=0.45 -0.04 0.38 rpy=0 0.261799387799 0, axis 0 0 0
- added joint l515_2_link_joint: type fixed, parent back_sensors, child l515_2_link, origin xyz=-0.045 0 0.185 rpy=0 -0.1745329252 0, axis 0 0 0
- added joint t265_link_joint: type fixed, parent back_sensors, child t265_link, origin xyz=0 0 0.095 rpy=0 0 0, axis 0 0 0

Commit message: stuff

File: ros/catkin_ws/src/david_config/urdf/david2.urdf (robot description, URDF)
Before this commit: robot david, 10 links, 9 joints
Links:
- added link t265_pose_frame
Joints:
- added joint t265_pose_joint: type fixed, parent t265_pose_frame, child base_link, origin xyz=0 0 -0.095 rpy=0 0 0, axis 0 0 0

Commit message: urdf

File: ros/catkin_ws/src/david_config/urdf/david2.urdf (robot description, URDF)
Before this commit: robot david, 11 links, 10 joints
Joints:
- joint d455_2_link_joint: origin xyz=-0.01 0.02 0.16 rpy=1.308996939 3.14159265 0 -> xyz=-0.01 0.02 0.16 rpy=0 3.14159265 0

Commit message: urdf

File: ros/catkin_ws/src/david_config/urdf/david2.urdf (robot description, URDF)
Before this commit: robot david, 11 links, 10 joints
Joints:
- joint d455_2_link_joint: origin xyz=-0.01 0.02 0.16 rpy=0 3.14159265 0 -> xyz=-0.01 0.02 0.16 rpy=-0.261799386 3.14159265 0

Commit message: urdf

File: ros/catkin_ws/src/david_config/urdf/david2.urdf (robot description, URDF)
Before this commit: robot david, 11 links, 10 joints
Joints:
- joint d455_2_link_joint: origin xyz=-0.01 0.02 0.16 rpy=-0.261799386 3.14159265 0 -> xyz=-0.01 0.02 0.16 rpy=-0.261799386 3.14159265 3.14159265

Commit message: mapping

File: ros/catkin_ws/src/david_config/urdf/david2.urdf (robot description, URDF)
Before this commit: robot david, 11 links, 10 joints
Joints:
- joint d455_2_link_joint: origin xyz=-0.01 0.02 0.16 rpy=-0.261799386 3.14159265 3.14159265 -> xyz=-0.01 0.02 0.16 rpy=0 -0.261799386 0

Commit message: mapping

File: ros/catkin_ws/src/david_config/urdf/david2.urdf (robot description, URDF)
Before this commit: robot david, 11 links, 10 joints
Joints:
- joint d455_2_link_joint: origin xyz=-0.01 0.02 0.16 rpy=0 -0.261799386 0 -> xyz=-0.01 0.02 0.16 rpy=0 0.261799386 -1.57

Commit message: mapping

File: ros/catkin_ws/src/david_config/urdf/david2.urdf (robot description, URDF)
Before this commit: robot david, 11 links, 10 joints
Joints:
- joint d455_1_link_joint: origin xyz=-0.005 -0.02 0.16 rpy=-1.8325957146 0 0 -> xyz=-0.005 -0.02 0.16 rpy=0 0.261799386 1.57

Commit message: mapping

File: ros/catkin_ws/src/david_config/urdf/david2.urdf (robot description, URDF)
Before this commit: robot david, 11 links, 10 joints
Joints:
- joint l515_2_link_joint: origin xyz=-0.045 0 0.185 rpy=0 -0.1745329252 0 -> xyz=-0.045 0 0.185 rpy=0 -0.1745329252 3.14

Commit message: mapping

File: ros/catkin_ws/src/david_config/urdf/david2.urdf (robot description, URDF)
Before this commit: robot david, 11 links, 10 joints
Joints:
- joint l515_2_link_joint: origin xyz=-0.045 0 0.185 rpy=0 -0.1745329252 3.14 -> xyz=-0.045 0 0.185 rpy=0 0.1745329252 3.14

Commit message: Update URDF

File: ros/catkin_ws/src/david_config/urdf/david2.urdf (robot description, URDF)
Before this commit: robot david, 11 links, 10 joints
Links:
- added link right_depth_plate_top
Joints:
- removed joint d455_2_link_joint
- added joint d455_2_joint: type fixed, parent right_depth_plate_top, child d455_2_link, origin xyz=0 -0.08265 -0.02027 rpy=0 0 0, axis 0 0 0
- added joint right_depth_plate_top_joint: type fixed, parent back_right, child right_depth_plate_top, origin xyz=0.4225 0.125 0.1651 rpy=0 0 0, axis 0 0 0

Commit message: Rotate d455_2_link correctly

File: ros/catkin_ws/src/david_config/urdf/david2.urdf (robot description, URDF)
Before this commit: robot david, 12 links, 11 joints
Joints:
- removed joint d455_2_joint
- added joint d455_2_link_joint: type fixed, parent right_depth_plate_top, child d455_2_link, origin xyz=0 -0.08265 -0.02027 rpy=0 0 -1.57, axis 0 0 0

Commit message: Update d455_1_link joint

File: ros/catkin_ws/src/david_config/urdf/david2.urdf (robot description, URDF)
Before this commit: robot david, 12 links, 11 joints
Joints:
- joint d455_1_link_joint: origin xyz=-0.005 -0.02 0.16 rpy=0 0.261799386 1.57 -> xyz=0.01 -0.01 0.28 rpy=0 0 1.57

Commit message: Change in Rear View Camera Angle

File: ros/catkin_ws/src/david_config/urdf/david2.urdf (robot description, URDF)
Before this commit: robot david, 12 links, 11 joints
Joints:
- joint l515_2_link_joint: origin xyz=-0.045 0 0.185 rpy=0 0.1745329252 3.14 -> xyz=-0.045 0 0.185 rpy=0 0.192 3.14

Commit message: Update urdf

File: ros/catkin_ws/src/david_config/urdf/david2.urdf (robot description, URDF)
Before this commit: robot david, 12 links, 11 joints
Joints:
- joint l515_2_link_joint: origin xyz=-0.045 0 0.185 rpy=0 0.192 3.14 -> xyz=-0.045 0 0.185 rpy=0  0.150 3.14

Commit message: stuff

File: ros/catkin_ws/src/david_config/urdf/david2.urdf (robot description, URDF)
Before this commit: robot david, 12 links, 11 joints
Joints:
- joint l515_2_link_joint: origin xyz=-0.045 0 0.185 rpy=0  0.150 3.14 -> xyz=-0.045 0 0.185 rpy=0 0.301 3.14

Commit message: Front Cam Angle Fix

File: ros/catkin_ws/src/david_config/urdf/david2.urdf (robot description, URDF)
Before this commit: robot david, 12 links, 11 joints
Joints:
- joint l515_1_link_joint: origin xyz=0.45 -0.04 0.38 rpy=0 0.261799387799 0 -> xyz=0.45 -0.04 0.38 rpy=0 0.28 0

Commit message: Update l515_1 angle

File: ros/catkin_ws/src/david_config/urdf/david2.urdf (robot description, URDF)
Before this commit: robot david, 12 links, 11 joints
Joints:
- joint l515_1_link_joint: origin xyz=0.45 -0.04 0.38 rpy=0 0.28 0 -> xyz=0.45 -0.04 0.38 rpy=0 0.352780229808 0

Commit message: Other direction

File: ros/catkin_ws/src/david_config/urdf/david2.urdf (robot description, URDF)
Before this commit: robot david, 12 links, 11 joints
Joints:
- joint l515_1_link_joint: origin xyz=0.45 -0.04 0.38 rpy=0 0.352780229808 0 -> xyz=0.45 -0.04 0.38 rpy=0 0.207219770192 0

Commit message: Try rotating t265_pose_joint to fix localization issue

File: ros/catkin_ws/src/david_config/urdf/david2.urdf (robot description, URDF)
Before this commit: robot david, 12 links, 11 joints
Joints:
- joint t265_pose_joint: origin xyz=0 0 -0.095 rpy=0 0 0 -> xyz=0 0 -0.095 rpy=0 0 3.1415926535

Commit message: Revert "Try rotating t265_pose_joint to fix localization issue"
This reverts commit f3cdbabeaf09597a865875866c937cf5c2c41bec.

File: ros/catkin_ws/src/david_config/urdf/david2.urdf (robot description, URDF)
Before this commit: robot david, 12 links, 11 joints
Joints:
- joint t265_pose_joint: origin xyz=0 0 -0.095 rpy=0 0 3.1415926535 -> xyz=0 0 -0.095 rpy=0 0 0

Commit message: urdf

File: ros/catkin_ws/src/david_config/urdf/david2.urdf (robot description, URDF)
Before this commit: robot david, 12 links, 11 joints
Joints:
- joint l515_2_link_joint: origin xyz=-0.045 0 0.185 rpy=0 0.301 3.14 -> xyz=-0.045 0 0.185 rpy=0 0.30 3.14
